Commit message: Comment out inertia spec for base_link

File: rc_model/urdf/rc_model.xacro (robot description, xacro)
@@ -5,9 +5,9 @@
   <xacro:include filename="$(find rc_model)/urdf/rc_model.gazebo" />
   <link name="base_link">
-    <inertial>
+    <!-- <inertial>
       <origin xyz="-1.3083309184741514e-15 0.12128943795441537 0.03369194136532842" rpy="0 0 0" />
       <mass value="1.3778870164240344" />
       <inertia ixx="0.005759" iyy="0.002706" izz="0.006735" ixy="-0.0" iyz="0.001087" ixz="-0.0" />
-    </inertial>
+    </inertial> -->
     <visual>
       <origin xyz="0 0 0" rpy="0 0 0" />

Commit message: Messing with collision geometry

File: rc_model/urdf/rc_model.xacro (robot description, xacro)
@@ -205,6 +205,9 @@
     <visual>
       <origin xyz="0.0685 -0.0025 0.003" rpy="0 0 0" />
-      <geometry>
+      <!-- <geometry>
         <mesh filename="package://rc_model/meshes/wheel_1.stl" scale="0.001 0.001 0.001" />
+      </geometry> -->
+      <geometry>
+        <box size="0.01 0.01 0.01" />
       </geometry>
       <material name="silver" />
@@ -277,5 +280,5 @@
     </collision>
   </link>
-  <link name="steering_rod_1">
+  <!-- <link name="steering_rod_1">
     <inertial>
       <origin xyz="-3.137386184182134e-13 1.734723475976807e-18 0.00824999999999997" rpy="0 0 0" />
@@ -298,6 +301,6 @@
       </geometry>
     </collision>
-  </link>
-  <link name="steering_bar_1">
+  </link> -->
+  <!-- <link name="steering_bar_1">
     <inertial>
       <origin xyz="-0.008747999625029047 -0.014067539563090594 -0.0015000000000000326" rpy="0 0 0" />
@@ -320,5 +323,5 @@
       </geometry>
     </collision>
-  </link>
+  </link> -->
   <joint name="servo_angle" type="revolute">
     <origin xyz="-0.015 0.0045 -0.018" rpy="0 0 0" />
@@ -395,10 +398,10 @@
     <axis xyz="1.0 -0.0 0.0" />
   </joint>
-  <joint name="Rigid 306" type="fixed">
+  <!-- <joint name="Rigid 306" type="fixed">
     <origin xyz="0.0 -0.02 -0.002" rpy="0 0 0" />
     <parent link="servo_horn_1" />
     <child link="steering_rod_1" />
-  </joint>
-  <joint name="Revolute 307" type="revolute">
+  </joint> -->
+  <!-- <joint name="Revolute 307" type="revolute">
     <origin xyz="0.0 0.0 0.0165" rpy="0 0 0" />
     <parent link="steering_rod_1" />
@@ -407,4 +410,4 @@
     <limit upper="0.488692" lower="-0.488692" effort="100" velocity="100" />
     <mimic joint="servo_angle" />
-  </joint>
+  </joint> -->
 </robot>

Commit message: Refactor joints and links to their own files

File: rc_model/urdf/rc_model.xacro (robot description, xacro)
@@ -4,410 +4,5 @@
   <xacro:include filename="$(find rc_model)/urdf/rc_model.trans" />
   <xacro:include filename="$(find rc_model)/urdf/rc_model.gazebo" />
-  <link name="base_link">
-    <!-- <inertial>
-      <origin xyz="-1.3083309184741514e-15 0.12128943795441537 0.03369194136532842" rpy="0 0 0" />
-      <mass value="1.3778870164240344" />
-      <inertia ixx="0.005759" iyy="0.002706" izz="0.006735" ixy="-0.0" iyz="0.001087" ixz="-0.0" />
-    </inertial> -->
-    <visual>
-      <origin xyz="0 0 0" rpy="0 0 0" />
-      <geometry>
-        <mesh filename="package://rc_model/meshes/base_link.stl"
-          scale="0.001 0.001 0.001" />
-      </geometry>
-      <material name="silver" />
-    </visual>
-    <collision>
-      <origin xyz="0 0 0" rpy="0 0 0" />
-      <geometry>
-        <mesh filename="package://rc_model/meshes/base_link.stl"
-          scale="0.001 0.001 0.001" />
-      </geometry>
-    </collision>
-  </link>
-  <link name="servo_horn_1">
-    <inertial>
-      <origin xyz="-1.460882973575682e-05 -0.007871889996444085 0.0006174758834835425" rpy="0 0 0" />
-      <mass value="0.00950784131380662" />
-      <inertia ixx="1e-06" iyy="0.0" izz="1e-06" ixy="-0.0" iyz="-0.0" ixz="0.0" />
-    </inertial>
-    <visual>
-      <origin xyz="-0.01 -0.0145 0.023" rpy="0 0 0" />
-      <geometry>
-        <mesh filename="package://rc_model/meshes/servo_horn_1.stl"
-          scale="0.001 0.001 0.001" />
-      </geometry>
-      <material name="silver" />
-    </visual>
-    <collision>
-      <origin xyz="-0.01 -0.0145 0.023" rpy="0 0 0" />
-      <geometry>
-        <mesh filename="package://rc_model/meshes/servo_horn_1.stl"
-          scale="0.001 0.001 0.001" />
-      </geometry>
-    </collision>
-  </link>
-  <link name="left_wheel_mount_1">
-    <inertial>
-      <origin xyz="0.0001100665752926111 -0.0003109939838788164 -0.00016990269857806864" rpy="0 0 0" />
-      <mass value="0.05436953130754834" />
-      <inertia ixx="7e-06" iyy="3e-06" izz="5e-06" ixy="-0.0" iyz="-0.0" ixz="-0.0" />
-    </inertial>
-    <visual>
-      <origin xyz="-0.064 -0.0025 0.003" rpy="0 0 0" />
-      <geometry>
-        <mesh filename="package://rc_model/meshes/left_wheel_mount_1.stl"
-          scale="0.001 0.001 0.001" />
-      </geometry>
-      <material name="silver" />
-    </visual>
-    <collision>
-      <origin xyz="-0.064 -0.0025 0.003" rpy="0 0 0" />
-      <geometry>
-        <mesh filename="package://rc_model/meshes/left_wheel_mount_1.stl"
-          scale="0.001 0.001 0.001" />
-      </geometry>
-    </collision>
-  </link>
-  <link name="right_wheel_mount_1">
-    <inertial>
-      <origin xyz="-0.00011006657149828514 -0.00031099398387884024 -0.00016990269874315057"
-        rpy="0 0 0" />
-      <mass value="0.05436953130754809" />
-      <inertia ixx="7e-06" iyy="3e-06" izz="5e-06" ixy="0.0" iyz="-0.0" ixz="0.0" />
-    </inertial>
-    <visual>
-      <origin xyz="0.064 -0.0025 0.003" rpy="0 0 0" />
-      <geometry>
-        <mesh filename="package://rc_model/meshes/right_wheel_mount_1.stl"
-          scale="0.001 0.001 0.001" />
-      </geometry>
-      <material name="silver" />
-    </visual>
-    <collision>
-      <origin xyz="0.064 -0.0025 0.003" rpy="0 0 0" />
-      <geometry>
-        <mesh filename="package://rc_model/meshes/right_wheel_mount_1.stl"
-          scale="0.001 0.001 0.001" />
-      </geometry>
-    </collision>
-  </link>
-  <link name="front_assembly_1">
-    <inertial>
-      <origin xyz="2.0263603307538467e-06 -0.013870173245129229 -0.010153618514841685" rpy="0 0 0" />
-      <mass value="0.5186122317437215" />
-      <inertia ixx="0.000468" iyy="0.000561" izz="0.000768" ixy="0.0" iyz="-0.000131" ixz="0.0" />
-    </inertial>
-    <visual>
-      <origin xyz="0.0 -0.0305 -0.02275" rpy="0 0 0" />
-      <geometry>
-        <mesh filename="package://rc_model/meshes/front_assembly_1.stl"
-          scale="0.001 0.001 0.001" />
-      </geometry>
-      <material name="silver" />
-    </visual>
-    <collision>
-      <origin xyz="0.0 -0.0305 -0.02275" rpy="0 0 0" />
-      <geometry>
-        <mesh filename="package://rc_model/meshes/front_assembly_1.stl"
-          scale="0.001 0.001 0.001" />
-      </geometry>
-    </collision>
-  </link>
-  <link name="suspension_axle_1">
-    <inertial>
-      <origin xyz="-3.669079600359632e-17 -0.03206500000000001 3.469446951953614e-18" rpy="0 0 0" />
-      <mass value="0.08896174562624065" />
-      <inertia ixx="3.2e-05" iyy="3e-06" izz="3.2e-05" ixy="-0.0" iyz="0.0" ixz="-0.0" />
-    </inertial>
-    <visual>
-      <origin xyz="-0.0 -0.09463 -0.02275" rpy="0 0 0" />
-      <geometry>
-        <mesh filename="package://rc_model/meshes/suspension_axle_1.stl"
-          scale="0.001 0.001 0.001" />
-      </geometry>
-      <material name="silver" />
-    </visual>
-    <collision>
-      <origin xyz="-0.0 -0.09463 -0.02275" rpy="0 0 0" />
-      <geometry>
-        <mesh filename="package://rc_model/meshes/suspension_axle_1.stl"
-          scale="0.001 0.001 0.001" />
-      </geometry>
-    </collision>
-  </link>
-  <link name="servo_1">
-    <inertial>
-      <origin xyz="-0.024893878005047748 0.0045000006838291935 0.010046478190773773" rpy="0 0 0" />
-      <mass value="0.24909707230016578" />
-      <inertia ixx="4e-05" iyy="6.7e-05" izz="4.3e-05" ixy="0.0" iyz="0.0" ixz="1e-06" />
-    </inertial>
-    <visual>
-      <origin xyz="-0.025 -0.01 0.005" rpy="0 0 0" />
-      <geometry>
-        <mesh filename="package://rc_model/meshes/servo_1.stl" scale="0.001 0.001 0.001" />
-      </geometry>
-      <material name="silver" />
-    </visual>
-    <collision>
-      <origin xyz="-0.025 -0.01 0.005" rpy="0 0 0" />
-      <geometry>
-        <mesh filename="package://rc_model/meshes/servo_1.stl" scale="0.001 0.001 0.001" />
-      </geometry>
-    </collision>
-  </link>
-  <link name="motor_1">
-    <inertial>
-      <origin xyz="-0.0245862223060676 0.00032401346399821285 -5.755815434930599e-06" rpy="0 0 0" />
-      <mass value="0.1278108358826081" />
-      <inertia ixx="2.3e-05" iyy="5.9e-05" izz="5.9e-05" ixy="-1e-06" iyz="-0.0" ixz="-0.0" />
-    </inertial>
-    <visual>
-      <origin xyz="-0.063 -0.18238 0.003" rpy="0 0 0" />
-      <geometry>
-        <mesh filename="package://rc_model/meshes/motor_1.stl" scale="0.001 0.001 0.001" />
-      </geometry>
-      <material name="silver" />
-    </visual>
-    <collision>
-      <origin xyz="-0.063 -0.18238 0.003" rpy="0 0 0" />
-      <geometry>
-        <mesh filename="package://rc_model/meshes/motor_1.stl" scale="0.001 0.001 0.001" />
-      </geometry>
-    </collision>
-  </link>
-  <link name="motor_2">
-    <inertial>
-      <origin xyz="0.024586222306067662 0.00032401346399821285 5.7558154691037845e-06" rpy="0 0 0" />
-      <mass value="0.1278108358826081" />
-      <inertia ixx="2.3e-05" iyy="5.9e-05" izz="5.9e-05" ixy="1e-06" iyz="0.0" ixz="-0.0" />
-    </inertial>
-    <visual>
-      <origin xyz="0.063 -0.18238 0.003" rpy="0 0 0" />
-      <geometry>
-        <mesh filename="package://rc_model/meshes/motor_2.stl" scale="0.001 0.001 0.001" />
-      </geometry>
-      <material name="silver" />
-    </visual>
-    <collision>
-      <origin xyz="0.063 -0.18238 0.003" rpy="0 0 0" />
-      <geometry>
-        <mesh filename="package://rc_model/meshes/motor_2.stl" scale="0.001 0.001 0.001" />
-      </geometry>
-    </collision>
-  </link>
-  <link name="wheel_1">
-    <inertial>
-      <origin xyz="-0.015146771015638341 1.0053778219838716e-06 -2.3198153083388295e-08" rpy="0 0 0" />
-      <mass value="0.569142071306609" />
-      <inertia ixx="0.001077" iyy="0.000616" izz="0.000616" ixy="-0.0" iyz="-0.0" ixz="-0.0" />
-    </inertial>
-    <visual>
-      <origin xyz="0.0685 -0.0025 0.003" rpy="0 0 0" />
-      <!-- <geometry>
-        <mesh filename="package://rc_model/meshes/wheel_1.stl" scale="0.001 0.001 0.001" />
-      </geometry> -->
-      <geometry>
-        <box size="0.01 0.01 0.01" />
-      </geometry>
-      <material name="silver" />
-    </visual>
-    <collision>
-      <origin xyz="0.0685 -0.0025 0.003" rpy="0 0 0" />
-      <geometry>
-        <mesh filename="package://rc_model/meshes/wheel_1.stl" scale="0.001 0.001 0.001" />
-      </geometry>
-    </collision>
-  </link>
-  <link name="wheel_2">
-    <inertial>
-      <origin xyz="0.015146771015638272 -1.00537782258929e-06 -2.319815317055815e-08" rpy="0 0 0" />
-      <mass value="0.569142071306609" />
-      <inertia ixx="0.001077" iyy="0.000616" izz="0.000616" ixy="-0.0" iyz="0.0" ixz="0.0" />
-    </inertial>
-    <visual>
-      <origin xyz="-0.0685 -0.0025 0.003" rpy="0 0 0" />
-      <geometry>
-        <mesh filename="package://rc_model/meshes/wheel_2.stl" scale="0.001 0.001 0.001" />
-      </geometry>
-      <material name="silver" />
-    </visual>
-    <collision>
-      <origin xyz="-0.0685 -0.0025 0.003" rpy="0 0 0" />
-      <geometry>
-        <mesh filename="package://rc_model/meshes/wheel_2.stl" scale="0.001 0.001 0.001" />
-      </geometry>
-    </collision>
-  </link>
-  <link name="wheel_3">
-    <inertial>
-      <origin xyz="-0.015146771015636287 1.00537782199428e-06 -2.3198136071388847e-08" rpy="0 0 0" />
-      <mass value="0.569142071306609" />
-      <inertia ixx="0.001077" iyy="0.000616" izz="0.000616" ixy="-0.0" iyz="-0.0" ixz="-0.0" />
-    </inertial>
-    <visual>
-      <origin xyz="0.0725 -0.18938 0.003" rpy="0 0 0" />
-      <geometry>
-        <mesh filename="package://rc_model/meshes/wheel_3.stl" scale="0.001 0.001 0.001" />
-      </geometry>
-      <material name="silver" />
-    </visual>
-    <collision>
-      <origin xyz="0.0725 -0.18938 0.003" rpy="0 0 0" />
-      <geometry>
-        <mesh filename="package://rc_model/meshes/wheel_3.stl" scale="0.001 0.001 0.001" />
-      </geometry>
-    </collision>
-  </link>
-  <link name="wheel_4">
-    <inertial>
-      <origin xyz="0.015146771015636287 -1.0053778232710364e-06 -2.319813606314891e-08" rpy="0 0 0" />
-      <mass value="0.569142071306609" />
-      <inertia ixx="0.001077" iyy="0.000616" izz="0.000616" ixy="-0.0" iyz="0.0" ixz="0.0" />
-    </inertial>
-    <visual>
-      <origin xyz="-0.0725 -0.18938 0.003" rpy="0 0 0" />
-      <geometry>
-        <mesh filename="package://rc_model/meshes/wheel_4.stl" scale="0.001 0.001 0.001" />
-      </geometry>
-      <material name="silver" />
-    </visual>
-    <collision>
-      <origin xyz="-0.0725 -0.18938 0.003" rpy="0 0 0" />
-      <geometry>
-        <mesh filename="package://rc_model/meshes/wheel_4.stl" scale="0.001 0.001 0.001" />
-      </geometry>
-    </collision>
-  </link>
-  <!-- <link name="steering_rod_1">
-    <inertial>
-      <origin xyz="-3.137386184182134e-13 1.734723475976807e-18 0.00824999999999997" rpy="0 0 0" />
-      <mass value="0.0009155582740264544" />
-      <inertia ixx="0.0" iyy="0.0" izz="0.0" ixy="0.0" iyz="-0.0" ixz="0.0" />
-    </inertial>
-    <visual>
-      <origin xyz="-0.01 0.0055 0.025" rpy="0 0 0" />
-      <geometry>
-        <mesh filename="package://rc_model/meshes/steering_rod_1.stl"
-          scale="0.001 0.001 0.001" />
-      </geometry>
-      <material name="silver" />
-    </visual>
-    <collision>
-      <origin xyz="-0.01 0.0055 0.025" rpy="0 0 0" />
-      <geometry>
-        <mesh filename="package://rc_model/meshes/steering_rod_1.stl"
-          scale="0.001 0.001 0.001" />
-      </geometry>
-    </collision>
-  </link> -->
-  <!-- <link name="steering_bar_1">
-    <inertial>
-      <origin xyz="-0.008747999625029047 -0.014067539563090594 -0.0015000000000000326" rpy="0 0 0" />
-      <mass value="0.018019633607194895" />
-      <inertia ixx="0.0" iyy="2.4e-05" izz="2.4e-05" ixy="-0.0" iyz="0.0" ixz="0.0" />
-    </inertial>
-    <visual>
-      <origin xyz="-0.01 0.0055 0.0085" rpy="0 0 0" />
-      <geometry>
-        <mesh filename="package://rc_model/meshes/steering_bar_1.stl"
-          scale="0.001 0.001 0.001" />
-      </geometry>
-      <material name="silver" />
-    </visual>
-    <collision>
-      <origin xyz="-0.01 0.0055 0.0085" rpy="0 0 0" />
-      <geometry>
-        <mesh filename="package://rc_model/meshes/steering_bar_1.stl"
-          scale="0.001 0.001 0.001" />
-      </geometry>
-    </collision>
-  </link> -->
-  <joint name="servo_angle" type="revolute">
-    <origin xyz="-0.015 0.0045 -0.018" rpy="0 0 0" />
-    <parent link="servo_1" />
-    <child link="servo_horn_1" />
-    <axis xyz="-0.0 -0.0 -1.0" />
-    <limit upper="0.488692" lower="-0.488692" effort="100" velocity="100" />
-  </joint>
-  <joint name="Revolute 275" type="revolute">
-    <origin xyz="0.064 -0.028 -0.02575" rpy="0 0 0" />
-    <parent link="front_assembly_1" />
-    <child link="left_wheel_mount_1" />
-    <axis xyz="-0.0 0.0 1.0" />
-    <limit upper="0.488692" lower="-0.488692" effort="100" velocity="100" />
-    <mimic joint="servo_angle" multiplier="-1" />
-  </joint>
-  <joint name="Revolute 276" type="revolute">
-    <origin xyz="-0.064 -0.028 -0.02575" rpy="0 0 0" />
-    <parent link="front_assembly_1" />
-    <child link="right_wheel_mount_1" />
-    <axis xyz="0.0 0.0 1.0" />
-    <limit upper="0.488692" lower="-0.488692" effort="100" velocity="100" />
-    <mimic joint="servo_angle" multiplier="-1" />
-  </joint>
-  <joint name="suspension" type="revolute">
-    <origin xyz="-0.0 -0.06413 0.0" rpy="0 0 0" />
-    <parent link="suspension_axle_1" />
-    <child link="front_assembly_1" />
-    <axis xyz="0.0 -1.0 0.0" />
-    <limit upper="0.069813" lower="-0.069813" effort="100" velocity="100" />
-  </joint>
-  <joint name="Rigid 278" type="fixed">
-    <origin xyz="0.0 0.09463 0.02275" rpy="0 0 0" />
-    <parent link="base_link" />
-    <child link="suspension_axle_1" />
-  </joint>
-  <joint name="Rigid 279" type="fixed">
-    <origin xyz="0.025 -0.0205 -0.02775" rpy="0 0 0" />
-    <parent link="front_assembly_1" />
-    <child link="servo_1" />
-  </joint>
-  <joint name="Rigid 280" type="fixed">
-    <origin xyz="0.063 0.18238 -0.003" rpy="0 0 0" />
-    <parent link="base_link" />
-    <child link="motor_1" />
-  </joint>
-  <joint name="Rigid 281" type="fixed">
-    <origin xyz="-0.063 0.18238 -0.003" rpy="0 0 0" />
-    <parent link="base_link" />
-    <child link="motor_2" />
-  </joint>
-  <joint name="front right wheel" type="continuous">
-    <origin xyz="-0.0045 0.0 0.0" rpy="0 0 0" />
-    <parent link="right_wheel_mount_1" />
-    <child link="wheel_1" />
-    <axis xyz="-1.0 -0.0 0.0" />
-  </joint>
-  <joint name="front left wheel" type="continuous">
-    <origin xyz="0.0045 0.0 0.0" rpy="0 0 0" />
-    <parent link="left_wheel_mount_1" />
-    <child link="wheel_2" />
-    <axis xyz="1.0 -0.0 -0.0" />
-  </joint>
-  <joint name="back right wheel" type="continuous">
-    <origin xyz="-0.0095 0.007 0.0" rpy="0 0 0" />
-    <parent link="motor_2" />
-    <child link="wheel_3" />
-    <axis xyz="-1.0 -0.0 0.0" />
-  </joint>
-  <joint name="back left wheel" type="continuous">
-    <origin xyz="0.0095 0.007 0.0" rpy="0 0 0" />
-    <parent link="motor_1" />
-    <child link="wheel_4" />
-    <axis xyz="1.0 -0.0 0.0" />
-  </joint>
-  <!-- <joint name="Rigid 306" type="fixed">
-    <origin xyz="0.0 -0.02 -0.002" rpy="0 0 0" />
-    <parent link="servo_horn_1" />
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