Commit message: Remove unused links

File: rc_model/urdf/links.xacro (robot description, xacro)
@@ -286,47 +286,3 @@
         </collision>
     </link>
-    <!-- <link name="steering_rod_1">
-        <inertial>
-          <origin xyz="-3.137386184182134e-13 1.734723475976807e-18 0.00824999999999997" rpy="0 0 0" />
-          <mass value="0.0009155582740264544" />
-          <inertia ixx="0.0" iyy="0.0" izz="0.0" ixy="0.0" iyz="-0.0" ixz="0.0" />
-        </inertial>
-        <visual>
-          <origin xyz="-0.01 0.0055 0.025" rpy="0 0 0" />
-          <geometry>
-            <mesh filename="package://rc_model/meshes/steering_rod_1.stl"
-              scale="0.001 0.001 0.001" />
-          </geometry>
-          <material name="silver" />
-        </visual>
-        <collision>
-          <origin xyz="-0.01 0.0055 0.025" rpy="0 0 0" />
-          <geometry>
-            <mesh filename="package://rc_model/meshes/steering_rod_1.stl"
-              scale="0.001 0.001 0.001" />
-          </geometry>
-        </collision>
-      </link> -->
-    <!-- <link name="steering_bar_1">
-        <inertial>
-          <origin xyz="-0.008747999625029047 -0.014067539563090594 -0.0015000000000000326" rpy="0 0 0" />
-          <mass value="0.018019633607194895" />
-          <inertia ixx="0.0" iyy="2.4e-05" izz="2.4e-05" ixy="-0.0" iyz="0.0" ixz="0.0" />
-        </inertial>
-        <visual>
-          <origin xyz="-0.01 0.0055 0.0085" rpy="0 0 0" />
-          <geometry>
-            <mesh filename="package://rc_model/meshes/steering_bar_1.stl"
-              scale="0.001 0.001 0.001" />
-          </geometry>
-          <material name="silver" />
-        </visual>
-        <collision>
-          <origin xyz="-0.01 0.0055 0.0085" rpy="0 0 0" />
-          <geometry>
-            <mesh filename="package://rc_model/meshes/steering_bar_1.stl"
-              scale="0.001 0.001 0.001" />
-          </geometry>
-        </collision>
-      </link> -->
 </robot>
