Commit message: Rename single-use stls

File: rc_model/urdf/joints.xacro (robot description, xacro)
@@ -3,6 +3,6 @@
     <joint name="servo_angle" type="revolute">
         <origin xyz="-0.015 0.0045 -0.018" rpy="0 0 0" />
-        <parent link="servo_1" />
-        <child link="servo_horn_1" />
+        <parent link="servo" />
+        <child link="servo_horn" />
         <axis xyz="-0.0 -0.0 -1.0" />
         <limit upper="0.488692" lower="-0.488692" effort="100" velocity="100" />
@@ -10,6 +10,6 @@
     <joint name="Revolute 275" type="revolute">
         <origin xyz="0.064 -0.028 -0.02575" rpy="0 0 0" />
-        <parent link="front_assembly_1" />
-        <child link="left_wheel_mount_1" />
+        <parent link="front_assembly" />
+        <child link="left_wheel_mount" />
         <axis xyz="-0.0 0.0 1.0" />
         <limit upper="0.488692" lower="-0.488692" effort="100" velocity="100" />
@@ -18,6 +18,6 @@
     <joint name="Revolute 276" type="revolute">
         <origin xyz="-0.064 -0.028 -0.02575" rpy="0 0 0" />
-        <parent link="front_assembly_1" />
-        <child link="right_wheel_mount_1" />
+        <parent link="front_assembly" />
+        <child link="right_wheel_mount" />
         <axis xyz="0.0 0.0 1.0" />
         <limit upper="0.488692" lower="-0.488692" effort="100" velocity="100" />
@@ -26,6 +26,6 @@
     <joint name="suspension" type="revolute">
         <origin xyz="-0.0 -0.06413 0.0" rpy="0 0 0" />
-        <parent link="suspension_axle_1" />
-        <child link="front_assembly_1" />
+        <parent link="suspension_axle" />
+        <child link="front_assembly" />
         <axis xyz="0.0 -1.0 0.0" />
         <limit upper="0.069813" lower="-0.069813" effort="100" velocity="100" />
@@ -34,10 +34,10 @@
         <origin xyz="0.0 0.09463 0.02275" rpy="0 0 0" />
         <parent link="base_link" />
-        <child link="suspension_axle_1" />
+        <child link="suspension_axle" />
     </joint>
     <joint name="Rigid 279" type="fixed">
         <origin xyz="0.025 -0.0205 -0.02775" rpy="0 0 0" />
-        <parent link="front_assembly_1" />
-        <child link="servo_1" />
+        <parent link="front_assembly" />
+        <child link="servo" />
     </joint>
     <joint name="Rigid 280" type="fixed">
@@ -53,5 +53,5 @@
     <joint name="front right wheel" type="continuous">
         <origin xyz="-0.0045 0.0 0.0" rpy="0 0 0" />
-        <parent link="right_wheel_mount_1" />
+        <parent link="right_wheel_mount" />
         <child link="wheel_1" />
         <axis xyz="-1.0 -0.0 0.0" />
@@ -59,5 +59,5 @@
     <joint name="front left wheel" type="continuous">
         <origin xyz="0.0045 0.0 0.0" rpy="0 0 0" />
-        <parent link="left_wheel_mount_1" />
+        <parent link="left_wheel_mount" />
         <child link="wheel_2" />
         <axis xyz="1.0 -0.0 -0.0" />
@@ -77,5 +77,5 @@
     <!-- <joint name="Rigid 306" type="fixed">
         <origin xyz="0.0 -0.02 -0.002" rpy="0 0 0" />
-        <parent link="servo_horn_1" />
+        <parent link="servo_horn" />
         <child link="steering_rod_1" />
       </joint> -->

File: rc_model/urdf/links.xacro (robot description, xacro)
@@ -23,5 +23,5 @@
         </collision>
     </link>
-    <link name="servo_horn_1">
+    <link name="servo_horn">
         <inertial>
             <origin xyz="-1.460882973575682e-05 -0.007871889996444085 0.0006174758834835425"
@@ -33,5 +33,5 @@
             <origin xyz="-0.01 -0.0145 0.023" rpy="0 0 0" />
             <geometry>
-                <mesh filename="package://rc_model/meshes/servo_horn_1.stl"
+                <mesh filename="package://rc_model/meshes/servo_horn.stl"
                     scale="0.001 0.001 0.001" />
             </geometry>
@@ -41,10 +41,10 @@
             <origin xyz="-0.01 -0.0145 0.023" rpy="0 0 0" />
             <geometry>
-                <mesh filename="package://rc_model/meshes/servo_horn_1.stl"
-                    scale="0.001 0.001 0.001" />
-            </geometry>
-        </collision>
-    </link>
-    <link name="left_wheel_mount_1">
+                <mesh filename="package://rc_model/meshes/servo_horn.stl"
+                    scale="0.001 0.001 0.001" />
+            </geometry>
+        </collision>
+    </link>
+    <link name="left_wheel_mount">
         <inertial>
             <origin xyz="0.0001100665752926111 -0.0003109939838788164 -0.00016990269857806864"
@@ -56,5 +56,5 @@
             <origin xyz="-0.064 -0.0025 0.003" rpy="0 0 0" />
             <geometry>
-                <mesh filename="package://rc_model/meshes/left_wheel_mount_1.stl"
+                <mesh filename="package://rc_model/meshes/left_wheel_mount.stl"
                     scale="0.001 0.001 0.001" />
             </geometry>
@@ -64,10 +64,10 @@
             <origin xyz="-0.064 -0.0025 0.003" rpy="0 0 0" />
             <geometry>
-                <mesh filename="package://rc_model/meshes/left_wheel_mount_1.stl"
-                    scale="0.001 0.001 0.001" />
-            </geometry>
-        </collision>
-    </link>
-    <link name="right_wheel_mount_1">
+                <mesh filename="package://rc_model/meshes/left_wheel_mount.stl"
+                    scale="0.001 0.001 0.001" />
+            </geometry>
+        </collision>
+    </link>
+    <link name="right_wheel_mount">
         <inertial>
             <origin xyz="-0.00011006657149828514 -0.00031099398387884024 -0.00016990269874315057"
@@ -79,5 +79,5 @@
             <origin xyz="0.064 -0.0025 0.003" rpy="0 0 0" />
             <geometry>
-                <mesh filename="package://rc_model/meshes/right_wheel_mount_1.stl"
+                <mesh filename="package://rc_model/meshes/right_wheel_mount.stl"
                     scale="0.001 0.001 0.001" />
             </geometry>
@@ -87,10 +87,10 @@
             <origin xyz="0.064 -0.0025 0.003" rpy="0 0 0" />
             <geometry>
-                <mesh filename="package://rc_model/meshes/right_wheel_mount_1.stl"
-                    scale="0.001 0.001 0.001" />
-            </geometry>
-        </collision>
-    </link>
-    <link name="front_assembly_1">
+                <mesh filename="package://rc_model/meshes/right_wheel_mount.stl"
+                    scale="0.001 0.001 0.001" />
+            </geometry>
+        </collision>
+    </link>
+    <link name="front_assembly">
         <inertial>
             <origin xyz="2.0263603307538467e-06 -0.013870173245129229 -0.010153618514841685"
@@ -103,5 +103,5 @@
             <origin xyz="0.0 -0.0305 -0.02275" rpy="0 0 0" />
             <geometry>
-                <mesh filename="package://rc_model/meshes/front_assembly_1.stl"
+                <mesh filename="package://rc_model/meshes/front_assembly.stl"
                     scale="0.001 0.001 0.001" />
             </geometry>
@@ -111,10 +111,10 @@
             <origin xyz="0.0 -0.0305 -0.02275" rpy="0 0 0" />
             <geometry>
-                <mesh filename="package://rc_model/meshes/front_assembly_1.stl"
-                    scale="0.001 0.001 0.001" />
-            </geometry>
-        </collision>
-    </link>
-    <link name="suspension_axle_1">
+                <mesh filename="package://rc_model/meshes/front_assembly.stl"
+                    scale="0.001 0.001 0.001" />
+            </geometry>
+        </collision>
+    </link>
+    <link name="suspension_axle">
         <inertial>
             <origin xyz="-3.669079600359632e-17 -0.03206500000000001 3.469446951953614e-18"
@@ -126,5 +126,5 @@
             <origin xyz="-0.0 -0.09463 -0.02275" rpy="0 0 0" />
             <geometry>
-                <mesh filename="package://rc_model/meshes/suspension_axle_1.stl"
+                <mesh filename="package://rc_model/meshes/suspension_axle.stl"
                     scale="0.001 0.001 0.001" />
             </geometry>
@@ -134,10 +134,10 @@
             <origin xyz="-0.0 -0.09463 -0.02275" rpy="0 0 0" />
             <geometry>
-                <mesh filename="package://rc_model/meshes/suspension_axle_1.stl"
-                    scale="0.001 0.001 0.001" />
-            </geometry>
-        </collision>
-    </link>
-    <link name="servo_1">
+                <mesh filename="package://rc_model/meshes/suspension_axle.stl"
+                    scale="0.001 0.001 0.001" />
+            </geometry>
+        </collision>
+    </link>
+    <link name="servo">
         <inertial>
             <origin xyz="-0.024893878005047748 0.0045000006838291935 0.010046478190773773"
@@ -149,5 +149,5 @@
             <origin xyz="-0.025 -0.01 0.005" rpy="0 0 0" />
             <geometry>
-                <mesh filename="package://rc_model/meshes/servo_1.stl" scale="0.001 0.001 0.001" />
+                <mesh filename="package://rc_model/meshes/servo.stl" scale="0.001 0.001 0.001" />
             </geometry>
             <material name="silver" />
@@ -156,5 +156,5 @@
             <origin xyz="-0.025 -0.01 0.005" rpy="0 0 0" />
             <geometry>
-                <mesh filename="package://rc_model/meshes/servo_1.stl" scale="0.001 0.001 0.001" />
+                <mesh filename="package://rc_model/meshes/servo.stl" scale="0.001 0.001 0.001" />
             </geometry>
         </collision>
@@ -211,9 +211,6 @@
         <visual>
             <origin xyz="0.0685 -0.0025 0.003" rpy="0 0 0" />
-            <!-- <geometry>
-            <mesh filename="package://rc_model/meshes/wheel_1.stl" scale="0.001 0.001 0.001" />
-          </geometry> -->
-            <geometry>
-                <box size="0.01 0.01 0.01" />
+            <geometry>
+                <mesh filename="package://rc_model/meshes/wheel_1.stl" scale="0.001 0.001 0.001" />
             </geometry>
             <material name="silver" />

Commit message: Update description to handle steer and speed control

File: rc_model/urdf/joints.xacro (robot description, xacro)
@@ -8,5 +8,5 @@
         <limit upper="0.488692" lower="-0.488692" effort="100" velocity="100" />
     </joint>
-    <joint name="Revolute 275" type="revolute">
+    <joint name="left_wheel_mount_turn" type="revolute">
         <origin xyz="0.064 -0.028 -0.02575" rpy="0 0 0" />
         <parent link="front_assembly" />
@@ -16,5 +16,5 @@
         <mimic joint="servo_angle" multiplier="-1" />
     </joint>
-    <joint name="Revolute 276" type="revolute">
+    <joint name="right_wheel_mount_turn" type="revolute">
         <origin xyz="-0.064 -0.028 -0.02575" rpy="0 0 0" />
         <parent link="front_assembly" />
@@ -51,5 +51,5 @@
         <child link="motor_2" />
     </joint>
-    <joint name="front right wheel" type="continuous">
+    <joint name="front_right_wheel" type="continuous">
         <origin xyz="-0.0045 0.0 0.0" rpy="0 0 0" />
         <parent link="right_wheel_mount" />
@@ -57,5 +57,5 @@
         <axis xyz="-1.0 -0.0 0.0" />
     </joint>
-    <joint name="front left wheel" type="continuous">
+    <joint name="front_left_wheel" type="continuous">
         <origin xyz="0.0045 0.0 0.0" rpy="0 0 0" />
         <parent link="left_wheel_mount" />
@@ -63,5 +63,5 @@
         <axis xyz="1.0 -0.0 -0.0" />
     </joint>
-    <joint name="back right wheel" type="continuous">
+    <joint name="back_right_wheel" type="continuous">
         <origin xyz="-0.0095 0.007 0.0" rpy="0 0 0" />
         <parent link="motor_2" />
@@ -69,5 +69,5 @@
         <axis xyz="-1.0 -0.0 0.0" />
     </joint>
-    <joint name="back left wheel" type="continuous">
+    <joint name="back_left_wheel" type="continuous">
         <origin xyz="0.0095 0.007 0.0" rpy="0 0 0" />
         <parent link="motor_1" />

Commit message: Add simplified wheel collision meshes and rename some

File: rc_model/urdf/joints.xacro (robot description, xacro)
@@ -44,33 +44,33 @@
         <origin xyz="0.063 0.18238 -0.003" rpy="0 0 0" />
         <parent link="base_link" />
-        <child link="motor_1" />
+        <child link="left_motor" />
     </joint>
     <joint name="Rigid 281" type="fixed">
         <origin xyz="-0.063 0.18238 -0.003" rpy="0 0 0" />
         <parent link="base_link" />
-        <child link="motor_2" />
+        <child link="right_motor" />
     </joint>
-    <joint name="front_right_wheel" type="continuous">
+    <joint name="front_right_wheel_joint" type="continuous">
         <origin xyz="-0.0045 0.0 0.0" rpy="0 0 0" />
         <parent link="right_wheel_mount" />
-        <child link="wheel_1" />
+        <child link="front_right_wheel" />
         <axis xyz="-1.0 -0.0 0.0" />
     </joint>
-    <joint name="front_left_wheel" type="continuous">
+    <joint name="front_left_wheel_joint" type="continuous">
         <origin xyz="0.0045 0.0 0.0" rpy="0 0 0" />
         <parent link="left_wheel_mount" />
-        <child link="wheel_2" />
+        <child link="front_left_wheel" />
         <axis xyz="1.0 -0.0 -0.0" />
     </joint>
-    <joint name="back_right_wheel" type="continuous">
+    <joint name="back_right_wheel_joint" type="continuous">
         <origin xyz="-0.0095 0.007 0.0" rpy="0 0 0" />
-        <parent link="motor_2" />
-        <child link="wheel_3" />
+        <parent link="right_motor" />
+        <child link="back_right_wheel" />
         <axis xyz="-1.0 -0.0 0.0" />
     </joint>
-    <joint name="back_left_wheel" type="continuous">
+    <joint name="back_left_wheel_joint" type="continuous">
         <origin xyz="0.0095 0.007 0.0" rpy="0 0 0" />
-        <parent link="motor_1" />
-        <child link="wheel_4" />
+        <parent link="left_motor" />
+        <child link="back_left_wheel" />
         <axis xyz="1.0 -0.0 0.0" />
     </joint>
@@ -78,10 +78,10 @@
         <origin xyz="0.0 -0.02 -0.002" rpy="0 0 0" />
         <parent link="servo_horn" />
-        <child link="steering_rod_1" />
+        <child link="steering_rod" />
       </joint> -->
     <!-- <joint name="Revolute 307" type="revolute">
         <origin xyz="0.0 0.0 0.0165" rpy="0 0 0" />
-        <parent link="steering_rod_1" />
-        <child link="steering_bar_1" />
+        <parent link="steering_rod" />
+        <child link="steering_bar" />
         <axis xyz="0.0 0.0 1.0" />
         <limit upper="0.488692" lower="-0.488692" effort="100" velocity="100" />

File: rc_model/urdf/links.xacro (robot description, xacro)
@@ -160,5 +160,5 @@
         </collision>
     </link>
-    <link name="motor_1">
+    <link name="left_motor">
         <inertial>
             <origin xyz="-0.0245862223060676 0.00032401346399821285 -5.755815434930599e-06"
@@ -170,5 +170,5 @@
             <origin xyz="-0.063 -0.18238 0.003" rpy="0 0 0" />
             <geometry>
-                <mesh filename="package://rc_model/meshes/motor_1.stl" scale="0.001 0.001 0.001" />
+                <mesh filename="package://rc_model/meshes/left_motor.stl" scale="0.001 0.001 0.001" />
             </geometry>
             <material name="silver" />
@@ -177,9 +177,9 @@
             <origin xyz="-0.063 -0.18238 0.003" rpy="0 0 0" />
             <geometry>
-                <mesh filename="package://rc_model/meshes/motor_1.stl" scale="0.001 0.001 0.001" />
-            </geometry>
-        </collision>
-    </link>
-    <link name="motor_2">
+                <mesh filename="package://rc_model/meshes/left_motor.stl" scale="0.001 0.001 0.001" />
+            </geometry>
+        </collision>
+    </link>
+    <link name="right_motor">
         <inertial>
             <origin xyz="0.024586222306067662 0.00032401346399821285 5.7558154691037845e-06"
@@ -191,5 +191,5 @@
             <origin xyz="0.063 -0.18238 0.003" rpy="0 0 0" />
             <geometry>
-                <mesh filename="package://rc_model/meshes/motor_2.stl" scale="0.001 0.001 0.001" />
+                <mesh filename="package://rc_model/meshes/right_motor.stl" scale="0.001 0.001 0.001" />
             </geometry>
             <material name="silver" />
@@ -198,9 +198,9 @@
             <origin xyz="0.063 -0.18238 0.003" rpy="0 0 0" />
             <geometry>
-                <mesh filename="package://rc_model/meshes/motor_2.stl" scale="0.001 0.001 0.001" />
-            </geometry>
-        </collision>
-    </link>
-    <link name="wheel_1">
+                <mesh filename="package://rc_model/meshes/right_motor.stl" scale="0.001 0.001 0.001" />
+            </geometry>
+        </collision>
+    </link>
+    <link name="front_right_wheel">
         <inertial>
             <origin xyz="-0.015146771015638341 1.0053778219838716e-06 -2.3198153083388295e-08"
@@ -212,5 +212,6 @@
             <origin xyz="0.0685 -0.0025 0.003" rpy="0 0 0" />
             <geometry>
-                <mesh filename="package://rc_model/meshes/wheel_1.stl" scale="0.001 0.001 0.001" />
+                <mesh filename="package://rc_model/meshes/front_right_wheel_collision.stl"
+                    scale="0.001 0.001 0.001" />
             </geometry>
             <material name="silver" />
@@ -219,9 +220,10 @@
             <origin xyz="0.0685 -0.0025 0.003" rpy="0 0 0" />
             <geometry>
-                <mesh filename="package://rc_model/meshes/wheel_1.stl" scale="0.001 0.001 0.001" />
-            </geometry>
-        </collision>
-    </link>
-    <link name="wheel_2">
+                <mesh filename="package://rc_model/meshes/front_right_wheel_collision.stl"
+                    scale="0.001 0.001 0.001" />
+            </geometry>
+        </collision>
+    </link>
+    <link name="front_left_wheel">
         <inertial>
             <origin xyz="0.015146771015638272 -1.00537782258929e-06 -2.319815317055815e-08"
@@ -233,5 +235,6 @@
             <origin xyz="-0.0685 -0.0025 0.003" rpy="0 0 0" />
             <geometry>
-                <mesh filename="package://rc_model/meshes/wheel_2.stl" scale="0.001 0.001 0.001" />
+                <mesh filename="package://rc_model/meshes/front_left_wheel_collision.stl"
+                    scale="0.001 0.001 0.001" />
             </geometry>
             <material name="silver" />
@@ -240,9 +243,10 @@
             <origin xyz="-0.0685 -0.0025 0.003" rpy="0 0 0" />
             <geometry>
-                <mesh filename="package://rc_model/meshes/wheel_2.stl" scale="0.001 0.001 0.001" />
-            </geometry>
-        </collision>
-    </link>
-    <link name="wheel_3">
+                <mesh filename="package://rc_model/meshes/front_left_wheel_collision.stl"
+                    scale="0.001 0.001 0.001" />
+            </geometry>
+        </collision>
+    </link>
+    <link name="back_right_wheel">
         <inertial>
             <origin xyz="-0.015146771015636287 1.00537782199428e-06 -2.3198136071388847e-08"
@@ -254,5 +258,6 @@
             <origin xyz="0.0725 -0.18938 0.003" rpy="0 0 0" />
             <geometry>
-                <mesh filename="package://rc_model/meshes/wheel_3.stl" scale="0.001 0.001 0.001" />
+                <mesh filename="package://rc_model/meshes/back_right_wheel_collision.stl"
+                    scale="0.001 0.001 0.001" />
             </geometry>
             <material name="silver" />
@@ -261,9 +266,10 @@
             <origin xyz="0.0725 -0.18938 0.003" rpy="0 0 0" />
             <geometry>
-                <mesh filename="package://rc_model/meshes/wheel_3.stl" scale="0.001 0.001 0.001" />
-            </geometry>
-        </collision>
-    </link>
-    <link name="wheel_4">
+                <mesh filename="package://rc_model/meshes/back_right_wheel_collision.stl"
+                    scale="0.001 0.001 0.001" />
+            </geometry>
+        </collision>
+    </link>
+    <link name="back_left_wheel">
         <inertial>
             <origin xyz="0.015146771015636287 -1.0053778232710364e-06 -2.319813606314891e-08"
@@ -275,5 +281,6 @@
             <origin xyz="-0.0725 -0.18938 0.003" rpy="0 0 0" />
             <geometry>
-                <mesh filename="package://rc_model/meshes/wheel_4.stl" scale="0.001 0.001 0.001" />
+                <mesh filename="package://rc_model/meshes/back_left_wheel_collision.stl"
+                    scale="0.001 0.001 0.001" />
             </geometry>
             <material name="silver" />
@@ -282,5 +289,6 @@
             <origin xyz="-0.0725 -0.18938 0.003" rpy="0 0 0" />
             <geometry>
-                <mesh filename="package://rc_model/meshes/wheel_4.stl" scale="0.001 0.001 0.001" />
+                <mesh filename="package://rc_model/meshes/back_left_wheel_collision.stl"
+                    scale="0.001 0.001 0.001" />
             </geometry>
         </collision>

Commit message: Add imu link

File: rc_model/urdf/joints.xacro (robot description, xacro)
@@ -30,4 +30,9 @@
         <axis xyz="0.0 -1.0 0.0" />
         <limit upper="0.069813" lower="-0.069813" effort="100" velocity="100" />
+    </joint>
+    <joint name="imu" type="fixed">
+        <origin xyz="0 0 0" rpy="0 0 0" />
+        <parent link="suspension_axle" />
+        <child link="imu_link" />
     </joint>
     <joint name="Rigid 278" type="fixed">

File: rc_model/urdf/links.xacro (robot description, xacro)
@@ -139,4 +139,6 @@
         </collision>
     </link>
+    <link name="imu_link">
+    </link>
     <link name="servo">
         <inertial>

Commit message: Add lidar scan to simulation

File: rc_model/urdf/joints.xacro (robot description, xacro)
@@ -35,4 +35,11 @@
         <parent link="suspension_axle" />
         <child link="imu_link" />
+    </joint>
+    <joint name="lidar_joint" type="fixed">
+        <!-- <axis xyz="0 1 0" /> -->
+        <!-- <origin xyz="0 0 ${height3 - axel_offset/2}" rpy="0 0 0"/> -->
+        <origin xyz="0 0 0" rpy="0 0 0" />
+        <parent link="suspension_axle"/>
+        <child link="lidar_link"/>
     </joint>
     <joint name="Rigid 278" type="fixed">

File: rc_model/urdf/links.xacro (robot description, xacro)
@@ -140,4 +140,12 @@
     </link>
     <link name="imu_link">
+        <!-- potentially need stuff here -->
+    </link>
+    <link name="lidar_link">
+        <!-- <collision>
+        <origin xyz="0 0 0" rpy="0 0 0"/>
+        <geometry>
+        <box size="0.1 0.1 0.1"/>
+        </geometry> -->
     </link>
     <link name="servo">

Commit message: Add simulated lidar

File: rc_model/urdf/joints.xacro (robot description, xacro)
@@ -39,6 +39,6 @@
         <!-- <axis xyz="0 1 0" /> -->
         <!-- <origin xyz="0 0 ${height3 - axel_offset/2}" rpy="0 0 0"/> -->
-        <origin xyz="0 0 0" rpy="0 0 0" />
-        <parent link="suspension_axle"/>
+        <origin xyz="0 0 0.075" rpy="0 0 0" />
+        <parent link="base_link"/>
         <child link="lidar_link"/>
     </joint>

File: rc_model/urdf/links.xacro (robot description, xacro)
@@ -148,4 +148,11 @@
         <box size="0.1 0.1 0.1"/>
         </geometry> -->
+        <visual>
+            <origin xyz="0 0 0" rpy="0 0 0" />
+            <geometry>
+                <box size="0.01 0.01 0.01" />
+            </geometry>
+            <material name="silver" />
+        </visual>
     </link>
     <link name="servo">
